Commit message: commit

File: urdf/Swirl.xacro (robot description, xacro)
@@ -1,7 +1,7 @@
 <?xml version="1.0" ?>
 <robot name="Swirl" xmlns:xacro="http://www.ros.org/wiki/xacro">
-<xacro:include filename="$(find Swirl_description)/urdf/materials.xacro" />
-<xacro:include filename="$(find Swirl_description)/urdf/Swirl.trans" />
-<xacro:include filename="$(find Swirl_description)/urdf/Swirl.gazebo" />
+<xacro:include filename="$(find swirlbot)/urdf/materials.xacro" />
+<xacro:include filename="$(find swirlbot)/urdf/Swirl.trans" />
+<xacro:include filename="$(find swirlbot)/urdf/Swirl.gazebo" />
 <link name="base_link">
   <inertial>
@@ -13,5 +13,5 @@
     <origin rpy="0 0 0" xyz="0 0 0"/>
     <geometry>
-      <mesh filename="package://Swirl_description/meshes/base_link.stl" scale="0.001 0.001 0.001"/>
+      <mesh filename="package://swirlbot/meshes/base_link.stl" scale="0.001 0.001 0.001"/>
     </geometry>
     <material name="silver"/>
@@ -20,5 +20,5 @@
     <origin rpy="0 0 0" xyz="0 0 0"/>
     <geometry>
-      <mesh filename="package://Swirl_description/meshes/base_link.stl" scale="0.001 0.001 0.001"/>
+      <mesh filename="package://swirlbot/meshes/base_link.stl" scale="0.001 0.001 0.001"/>
     </geometry>
   </collision>
@@ -33,5 +33,5 @@
     <origin rpy="0 0 0" xyz="-0.150737 -0.049393 0.229787"/>
     <geometry>
-      <mesh filename="package://Swirl_description/meshes/wheel_shaft_1.stl" scale="0.001 0.001 0.001"/>
+      <mesh filename="package://swirlbot/meshes/wheel_shaft_1.stl" scale="0.001 0.001 0.001"/>
     </geometry>
     <material name="silver"/>
@@ -40,5 +40,5 @@
     <origin rpy="0 0 0" xyz="-0.150737 -0.049393 0.229787"/>
     <geometry>
-      <mesh filename="package://Swirl_description/meshes/wheel_shaft_1.stl" scale="0.001 0.001 0.001"/>
+      <mesh filename="package://swirlbot/meshes/wheel_shaft_1.stl" scale="0.001 0.001 0.001"/>
     </geometry>
   </collision>
@@ -53,5 +53,5 @@
     <origin rpy="0 0 0" xyz="-0.600737 -0.049393 0.229787"/>
     <geometry>
-      <mesh filename="package://Swirl_description/meshes/wheel_shaft_3.stl" scale="0.001 0.001 0.001"/>
+      <mesh filename="package://swirlbot/meshes/wheel_shaft_3.stl" scale="0.001 0.001 0.001"/>
     </geometry>
     <material name="silver"/>
@@ -60,5 +60,5 @@
     <origin rpy="0 0 0" xyz="-0.600737 -0.049393 0.229787"/>
     <geometry>
-      <mesh filename="package://Swirl_description/meshes/wheel_shaft_3.stl" scale="0.001 0.001 0.001"/>
+      <mesh filename="package://swirlbot/meshes/wheel_shaft_3.stl" scale="0.001 0.001 0.001"/>
     </geometry>
   </collision>
@@ -73,5 +73,5 @@
     <origin rpy="0 0 0" xyz="-0.600737 -0.499393 0.229787"/>
     <geometry>
-      <mesh filename="package://Swirl_description/meshes/wheel_shaft_4.stl" scale="0.001 0.001 0.001"/>
+      <mesh filename="package://swirlbot/meshes/wheel_shaft_4.stl" scale="0.001 0.001 0.001"/>
     </geometry>
     <material name="silver"/>
@@ -80,5 +80,5 @@
     <origin rpy="0 0 0" xyz="-0.600737 -0.499393 0.229787"/>
     <geometry>
-      <mesh filename="package://Swirl_description/meshes/wheel_shaft_4.stl" scale="0.001 0.001 0.001"/>
+      <mesh filename="package://swirlbot/meshes/wheel_shaft_4.stl" scale="0.001 0.001 0.001"/>
     </geometry>
   </collision>
@@ -93,5 +93,5 @@
     <origin rpy="0 0 0" xyz="-0.150737 -0.499393 0.229787"/>
     <geometry>
-      <mesh filename="package://Swirl_description/meshes/wheel_shaft_2.stl" scale="0.001 0.001 0.001"/>
+      <mesh filename="package://swirlbot/meshes/wheel_shaft_2.stl" scale="0.001 0.001 0.001"/>
     </geometry>
     <material name="silver"/>
@@ -100,5 +100,5 @@
     <origin rpy="0 0 0" xyz="-0.150737 -0.499393 0.229787"/>
     <geometry>
-      <mesh filename="package://Swirl_description/meshes/wheel_shaft_2.stl" scale="0.001 0.001 0.001"/>
+      <mesh filename="package://swirlbot/meshes/wheel_shaft_2.stl" scale="0.001 0.001 0.001"/>
     </geometry>
   </collision>
@@ -113,5 +113,5 @@
     <origin rpy="0 0 0" xyz="-0.422715 -0.958785 0.851169"/>
     <geometry>
-      <mesh filename="package://Swirl_description/meshes/wheel_2.stl" scale="0.001 0.001 0.001"/>
+      <mesh filename="package://swirlbot/meshes/wheel_2.stl" scale="0.001 0.001 0.001"/>
     </geometry>
     <material name="silver"/>
@@ -120,5 +120,5 @@
     <origin rpy="0 0 0" xyz="-0.422715 -0.958785 0.851169"/>
     <geometry>
-      <mesh filename="package://Swirl_description/meshes/wheel_2.stl" scale="0.001 0.001 0.001"/>
+      <mesh filename="package://swirlbot/meshes/wheel_2.stl" scale="0.001 0.001 0.001"/>
     </geometry>
   </collision>
@@ -133,5 +133,5 @@
     <origin rpy="0 0 0" xyz="-0.422715 -0.058785 0.851169"/>
     <geometry>
-      <mesh filename="package://Swirl_description/meshes/wheel_1.stl" scale="0.001 0.001 0.001"/>
+      <mesh filename="package://swirlbot/meshes/wheel_1.stl" scale="0.001 0.001 0.001"/>
     </geometry>
     <material name="silver"/>
@@ -140,5 +140,5 @@
     <origin rpy="0 0 0" xyz="-0.422715 -0.058785 0.851169"/>
     <geometry>
-      <mesh filename="package://Swirl_description/meshes/wheel_1.stl" scale="0.001 0.001 0.001"/>
+      <mesh filename="package://swirlbot/meshes/wheel_1.stl" scale="0.001 0.001 0.001"/>
     </geometry>
   </collision>
@@ -153,5 +153,5 @@
     <origin rpy="0 0 0" xyz="-1.212715 -0.058785 0.851169"/>
     <geometry>
-      <mesh filename="package://Swirl_description/meshes/wheel_3.stl" scale="0.001 0.001 0.001"/>
+      <mesh filename="package://swirlbot/meshes/wheel_3.stl" scale="0.001 0.001 0.001"/>
     </geometry>
     <material name="silver"/>
@@ -160,5 +160,5 @@
     <origin rpy="0 0 0" xyz="-1.212715 -0.058785 0.851169"/>
     <geometry>
-      <mesh filename="package://Swirl_description/meshes/wheel_3.stl" scale="0.001 0.001 0.001"/>
+      <mesh filename="package://swirlbot/meshes/wheel_3.stl" scale="0.001 0.001 0.001"/>
     </geometry>
   </collision>
@@ -173,5 +173,5 @@
     <origin rpy="0 0 0" xyz="-1.212715 -0.958785 0.851169"/>
     <geometry>
-      <mesh filename="package://Swirl_description/meshes/wheel_4.stl" scale="0.001 0.001 0.001"/>
+      <mesh filename="package://swirlbot/meshes/wheel_4.stl" scale="0.001 0.001 0.001"/>
     </geometry>
     <material name="silver"/>
@@ -180,5 +180,5 @@
     <origin rpy="0 0 0" xyz="-1.212715 -0.958785 0.851169"/>
     <geometry>
-      <mesh filename="package://Swirl_description/meshes/wheel_4.stl" scale="0.001 0.001 0.001"/>
+      <mesh filename="package://swirlbot/meshes/wheel_4.stl" scale="0.001 0.001 0.001"/>
     </geometry>
   </collision>
@@ -193,5 +193,5 @@
     <origin rpy="0 0 0" xyz="-0.150737 -0.049393 0.179787"/>
     <geometry>
-      <mesh filename="package://Swirl_description/meshes/wheel_link_1.stl" scale="0.001 0.001 0.001"/>
+      <mesh filename="package://swirlbot/meshes/wheel_link_1.stl" scale="0.001 0.001 0.001"/>
     </geometry>
     <material name="silver"/>
@@ -200,5 +200,5 @@
     <origin rpy="0 0 0" xyz="-0.150737 -0.049393 0.179787"/>
     <geometry>
-      <mesh filename="package://Swirl_description/meshes/wheel_link_1.stl" scale="0.001 0.001 0.001"/>
+      <mesh filename="package://swirlbot/meshes/wheel_link_1.stl" scale="0.001 0.001 0.001"/>
     </geometry>
   </collision>
@@ -213,5 +213,5 @@
     <origin rpy="0 0 0" xyz="-0.600737 -0.049393 0.179787"/>
     <geometry>
-      <mesh filename="package://Swirl_description/meshes/wheel_link_3.stl" scale="0.001 0.001 0.001"/>
+      <mesh filename="package://swirlbot/meshes/wheel_link_3.stl" scale="0.001 0.001 0.001"/>
     </geometry>
     <material name="silver"/>
@@ -220,5 +220,5 @@
     <origin rpy="0 0 0" xyz="-0.600737 -0.049393 0.179787"/>
     <geometry>
-      <mesh filename="package://Swirl_description/meshes/wheel_link_3.stl" scale="0.001 0.001 0.001"/>
+      <mesh filename="package://swirlbot/meshes/wheel_link_3.stl" scale="0.001 0.001 0.001"/>
     </geometry>
   </collision>
@@ -233,5 +233,5 @@
     <origin rpy="0 0 0" xyz="-0.600737 -0.499393 0.179787"/>
     <geometry>
-      <mesh filename="package://Swirl_description/meshes/wheel_link_4.stl" scale="0.001 0.001 0.001"/>
+      <mesh filename="package://swirlbot/meshes/wheel_link_4.stl" scale="0.001 0.001 0.001"/>
     </geometry>
     <material name="silver"/>
@@ -240,5 +240,5 @@
     <origin rpy="0 0 0" xyz="-0.600737 -0.499393 0.179787"/>
     <geometry>
-      <mesh filename="package://Swirl_description/meshes/wheel_link_4.stl" scale="0.001 0.001 0.001"/>
+      <mesh filename="package://swirlbot/meshes/wheel_link_4.stl" scale="0.001 0.001 0.001"/>
     </geometry>
   </collision>
@@ -253,5 +253,5 @@
     <origin rpy="0 0 0" xyz="-0.150737 -0.499393 0.179787"/>
     <geometry>
-      <mesh filename="package://Swirl_description/meshes/wheel_link_2.stl" scale="0.001 0.001 0.001"/>
+      <mesh filename="package://swirlbot/meshes/wheel_link_2.stl" scale="0.001 0.001 0.001"/>
     </geometry>
     <material name="silver"/>
@@ -260,5 +260,5 @@
     <origin rpy="0 0 0" xyz="-0.150737 -0.499393 0.179787"/>
     <geometry>
-      <mesh filename="package://Swirl_description/meshes/wheel_link_2.stl" scale="0.001 0.001 0.001"/>
+      <mesh filename="package://swirlbot/meshes/wheel_link_2.stl" scale="0.001 0.001 0.001"/>
     </geometry>
   </collision>
